Commit message: remove cameras for now to make local costmap look right

File: porter_bot_description/src/description/porter_bot_description.urdf (robot description, URDF)
Before this commit: robot porter_bot, 6 links, 5 joints
Links:
- removed link camera_depth_frame
- removed link camera_link
- link lidar_link: mass 0.125 -> 0.1; geometry collision cylinder length=0.035 radius=0.0308; visual cylinder length=0.055 radius=0.0508
Joints:
- removed joint camera_depth_joint
- removed joint camera_joint
- joint lidar_joint: origin xyz=0 0 0.12 rpy=0 0 0 -> xyz=0 0 0.32 rpy=0 0 0

File: porter_bot_description/src/description/robot_description/porter_bot_no_xacro.urdf (robot description, URDF)
Before this commit: robot porter_bot, 10 links, 9 joints
Links:
- removed link camera_depth_frame
- removed link camera_link
- link lidar_link: mass 0.125 -> 0.1; geometry collision cylinder length=0.035 radius=0.0308; visual cylinder length=0.055 radius=0.0508
Joints:
- removed joint camera_depth_joint
- removed joint camera_joint
- joint lidar_joint: origin xyz=0 0 0.12 rpy=0 0 0 -> xyz=0 0 0.32 rpy=0 0 0
