Commit message: use default model from tutorials to test controls

File: src/porter_bot_description/src/description/porter_bot_description.urdf (robot description, URDF)
Before this commit: robot porter_bot, 4 links, 3 joints
Links:
- added link caster_wheel; visual sphere radius=0.02
Joints:
- added joint caster_wheel_joint: type fixed, parent base_link, child caster_wheel, origin xyz=0.05 0 -0.04 rpy=0 0 0

File: src/porter_bot_description/src/description/porter_bot_description_expanded.urdf (robot description, URDF)
Before this commit: robot porter_bot, 8 links, 7 joints
Links:
- removed link frontwhl_l_link
- removed link frontwhl_r_link
- added link caster_wheel; visual sphere radius=0.02
- link rearwhl_l_link: mass 0.5 -> 0.2
- link rearwhl_r_link: mass 0.5 -> 0.2
Joints:
- removed joint frontwhl_l_joint
- removed joint frontwhl_r_joint
- added joint caster_wheel_joint: type fixed, parent base_link, child caster_wheel, origin xyz=0.05 0 -0.04 rpy=0 0 0
