Commit message: caster and footprint
added caster and footprint

File: src/porter_bot_description/src/description/robot_description/porter_bot.urdf (robot description, URDF)
Before this commit: robot porter_bot, 3 links, 2 joints
Links:
- added link base_footprint_link
- added link caster_wheel_link; visual sphere radius=0.05
Joints:
- added joint base_caster_wheel_joint: type fixed, parent base_link, child caster_wheel_link, origin xyz=0.2 0 -0.05 rpy=0 0 0
- added joint base_joint: type fixed, parent base_footprint_link, child base_link, origin xyz=0 0 -0.1 rpy=0 0 0
