Commit message: inertias
sphere and cylinder inertias

File: src/porter_bot_description/src/description/robot_description/common_properties.xacro (robot description, xacro)
@@ -1,5 +1,5 @@
 <?xml version="1.0"?>
 <robot xmlns:xacro="http://wwww.ros.org/wiki/xacro">
- <material name="green">
+    <material name="green">
         <color rgba="0.5 0 0 1" />
     </material>
@@ -7,3 +7,30 @@
         <color rgba="0.5 0.5 0.5 1" />
     </material>
+    <xacro:macro name="box_inertia" params="m l w h xyz rpy">
+        <inertial>
+            <origin xyz="${xyz}" rpy="${rpy}" />
+            <mass value="${m}" />
+            <inertia ixx="${(m/12) * (h*h + l*l)}" ixy="0" ixz="0"
+                     iyy="${(m/12) * (w*w + l*l)}" iyz="0"
+                     izz="${(m/12) * (w*w + h*h)}" />
+        </inertial>
+    </xacro:macro>
+    <xacro:macro name="sphere_inertia" params="m r xyz rpy">
+        <inertial>
+            <origin xyz="${xyz}" rpy="${rpy}" />
+            <mass value="${m}" />
+            <inertia ixx="${(2/5) * (m * r*r)}" ixy="0" ixz="0"
+                     iyy="${(2/5) * (m * r*r)}" iyz="0"
+                     izz="${(2/5) * (m * r*r)}" />
+        </inertial>
+    </xacro:macro>
+    <xacro:macro name="cylinder_inertia" params="m r h xyz rpy">
+        <inertial>
+            <origin xyz="${xyz}" rpy="${rpy}" />
+            <mass value="${m}" />
+            <inertia ixx="${(1/12) * m * ((3 * r*r) + (h * h))}" ixy="0" ixz="0"
+                     iyy="${(1/12) * m * ((3 * r*r) + (h * h))}" iyz="0"
+                     izz="${(1/2) * (m * r*r)}" />
+        </inertial>
+    </xacro:macro>
 </robot>

File: src/porter_bot_description/src/description/robot_description/mobile_base.xacro (robot description, xacro)
@@ -15,4 +15,6 @@
                 <material name="grey" />
             </visual>
+            <xacro:cylinder_inertia m="0.05" r="${wheel_radius}" h="${wheel_length}"
+                            xyz="0 0 0}" rpy="0 0 0" />
         </link>
     </xacro:macro>
@@ -27,4 +29,6 @@
             <material name="green" />
         </visual>
+        <xacro:box_inertia m="5.0" l="${base_length}" w="${base_width}" h="${base_height}"
+                            xyz="0 0 ${base_height / 2.0}" rpy="0 0 0" />
     </link>
     <xacro:wheel_link prefix="right" />
@@ -39,6 +43,8 @@
             <material name="grey" />
         </visual>
+        <xacro:sphere_inertia m="1.0" r="${wheel_radius / 2.0}"
+                            xyz="0 0 0}" rpy="0 0 0" />
     </link>
-     <link name="base_footprint_link">
+    <link name="base_footprint_link">
     </link>
     <joint name="base_right_wheel_joint" type="continuous">

Commit message: fix intertias

File: src/porter_bot_description/src/description/robot_description/common_properties.xacro (robot description, xacro)
@@ -29,7 +29,7 @@
             <origin xyz="${xyz}" rpy="${rpy}" />
             <mass value="${m}" />
-            <inertia ixx="${(1/12) * m * ((3 * r*r) + (h * h))}" ixy="0" ixz="0"
-                     iyy="${(1/12) * m * ((3 * r*r) + (h * h))}" iyz="0"
-                     izz="${(1/2) * (m * r*r)}" />
+            <inertia ixx="${(m/12) * ((3 * r*r) + (h * h))}" ixy="0" ixz="0"
+                     iyy="${(m/12) * ((3 * r*r) + (h * h))}" iyz="0"
+                     izz="${(m/2) * (r*r)}" />
         </inertial>
     </xacro:macro>

File: src/porter_bot_description/src/description/robot_description/mobile_base.xacro (robot description, xacro)
@@ -15,6 +15,12 @@
                 <material name="grey" />
             </visual>
-            <xacro:cylinder_inertia m="0.05" r="${wheel_radius}" h="${wheel_length}"
-                            xyz="0 0 0}" rpy="0 0 0" />
+            <collision>
+                <geometry>
+                    <cylinder radius="${wheel_radius}" length="${wheel_length}" />
+                </geometry>
+                <origin xyz="0 0 0" rpy="${pi / 2.0} 0 0" />
+            </collision>
+            <xacro:cylinder_inertia m="1.0" r="${wheel_radius}" h="${wheel_length}"
+                                    xyz="0 0 0" rpy="${pi / 2.0} 0 0" />
         </link>
     </xacro:macro>
@@ -29,4 +35,10 @@
             <material name="green" />
         </visual>
+        <collision>
+            <geometry>
+                <box size="${base_length} ${base_width} ${base_height}" />
+            </geometry>
+            <origin xyz="0 0 ${base_height / 2.0}" rpy="0 0 0" />
+        </collision>
         <xacro:box_inertia m="5.0" l="${base_length}" w="${base_width}" h="${base_height}"
                             xyz="0 0 ${base_height / 2.0}" rpy="0 0 0" />
@@ -43,6 +55,12 @@
             <material name="grey" />
         </visual>
-        <xacro:sphere_inertia m="1.0" r="${wheel_radius / 2.0}"
-                            xyz="0 0 0}" rpy="0 0 0" />
+        <collision>
+            <geometry>
+                <sphere radius="${wheel_radius / 2.0}" />
+            </geometry>
+            <origin xyz="0 0 0" rpy="0 0 0" />
+        </collision>
+        <xacro:sphere_inertia m="0.5" r="${wheel_radius / 2.0}"
+                                xyz="0 0 0" rpy="0 0 0" />
     </link>
     <link name="base_footprint_link">

Commit message: arm module
arm module definition

File: src/porter_bot_description/src/description/robot_description/common_properties.xacro (robot description, xacro)
@@ -6,4 +6,10 @@
      <material name="grey">
         <color rgba="0.5 0.5 0.5 1" />
+    </material>
+    <material name="orange">
+        <color rgba="1.0 0.5 0 1" />
+    </material>
+    <material name="yellow">
+        <color rgba="1.0 1.0 0 1" />
     </material>
     <xacro:macro name="box_inertia" params="m l w h xyz rpy">
