Commit message: added arm xacro
arm definition and materials

File: src/porter_bot_description/src/description/robot_description/arm.xacro (robot description, xacro)
@@ -16,4 +16,12 @@
             <material name="orange" />
         </visual>
+        <collision>
+            <geometry>
+                <box size="${arm_base_length} ${arm_base_width} ${arm_base_height}" />
+            </geometry>
+            <origin xyz="0 0 ${arm_base_height / 2.0}" rpy="0 0 0" />
+        </collision>
+        <xacro:box_inertia m="0.5" l="${2 * arm_base_length}" w="${2 * arm_base_width}" h="${2*arm_base_height}"
+                            xyz="0 0 ${arm_base_height / 2.0}" rpy="0 0 0"/>
     </link>
     <link name="forearm_link" >
@@ -25,4 +33,12 @@
             <material name="yellow" />
         </visual>
+        <collision>
+            <geometry>
+                <cylinder radius="${forearm_radius}" length="${forearm_length}" />
+            </geometry>
+            <origin xyz="0 0 ${forearm_length / 2.0}" rpy="0 0 0" />
+        </collision>
+        <xacro:cylinder_inertia m="0.3" r="${2 * forearm_radius}" h="${2 * forearm_length}"
+                                xyz="0 0 ${forearm_length / 2.0}" rpy="0 0 0" />
     </link>
     <link name="hand_link" >
@@ -31,7 +47,15 @@
                 <cylinder radius="${hand_radius}" length="${hand_length}" />
             </geometry>
-            <origin xyz="0 0 ${forearm_length / 2.0}" rpy="0 0 0" />
+            <origin xyz="0 0 ${hand_length / 2.0}" rpy="0 0 0" />
             <material name="orange" />
         </visual>
+        <collision>
+            <geometry>
+                <cylinder radius="${hand_radius}" length="${hand_length}" />
+            </geometry>
+            <origin xyz="0 0 ${hand_length / 2.0}" rpy="0 0 0" />
+        </collision>
+         <xacro:cylinder_inertia m="0.3" r="${2*hand_radius}" h="${2*hand_length}"
+                                xyz="0 0 ${hand_length / 2.0}" rpy="0 0 0" />
     </link>
     <joint name="arm_base_forearm_joint" type="revolute">
@@ -41,4 +65,5 @@
         <axis xyz="0 1 0"/>
         <limit lower="0" upper="${pi/2}" effort="100" velocity="100" />
+        <dynamics friction="0.05" damping="0.1" />
     </joint>
     <joint name="forearm_hand_joint" type="revolute">
@@ -48,4 +73,5 @@
         <axis xyz="0 1 0"/>
         <limit lower="0" upper="${pi/2}" effort="100" velocity="100" />
+        <dynamics friction="0.05" damping="0.1" />
     </joint>
 </robot>

File: src/porter_bot_description/src/description/robot_description/standalone_arm.urdf.xacro (robot description, xacro)
@@ -3,3 +3,4 @@
     <xacro:include filename="$(find porter_bot_description)/src/description/robot_description/common_properties.xacro" />
      <xacro:include filename="$(find porter_bot_description)/src/description/robot_description/arm.xacro" />
+      <xacro:include filename="$(find porter_bot_description)/src/description/robot_description/arm_gazebo.xacro" />
 </robot>
