Commit message: xacro
variables for the urdf

File: src/porter_bot_description/src/description/robot_description/porter_bot.urdf.xacro (robot description, xacro)
@@ -1,4 +1,9 @@
 <?xml version="1.0"?>
-<robot name="porter_bot">
+<robot name="porter_bot" xmlns:xacro="http://wwww.ros.org/wiki/xacro">
+    <xacro:property name="base_length" value="0.6" />
+    <xacro:property name="base_width" value="0.4" />
+    <xacro:property name="base_height" value="0.2" />
+    <xacro:property name="wheel_radius" value="0.1" />
+    <xacro:property name="wheel_length" value="0.05" />
     <material name="green">
         <color rgba="0.5 0 0 1" />
@@ -11,8 +16,8 @@
             <geometry>
                 <!--  <box size="0.157 0.073 0.055" />  -->
-                <box size="0.6 0.4 0.2" />
+                <box size="${base_length} ${base_width} ${base_height}" />
             </geometry>
             <!--  <origin xyz="0 0 0.0275" rpy="0 0 0" /> -->
-            <origin xyz="0 0 0.1" rpy="0 0 0" />
+            <origin xyz="0 0 ${base_height / 2.0}" rpy="0 0 0" />
             <material name="green" />
         </visual>
@@ -22,7 +27,7 @@
             <geometry>
                 <!-- <cylinder radius="0.03" length="0.007" /> -->
-                <cylinder radius="0.1" length="0.05" />
+                <cylinder radius="${wheel_radius}" length="${wheel_length}" />
             </geometry>
-            <origin xyz="0 0 0" rpy="1.57 0 0" />
+            <origin xyz="0 0 0" rpy="${pi / 2.0} 0 0" />
             <material name="grey" />
         </visual>
@@ -32,7 +37,7 @@
             <geometry>
                 <!-- <cylinder radius="0.03" length="0.007" /> -->
-                <cylinder radius="0.1" length="0.05" />
+                <cylinder radius="${wheel_radius}" length="${wheel_length}" />
             </geometry>
-            <origin xyz="0 0 0" rpy="1.57 0 0" />
+            <origin xyz="0 0 0" rpy="${pi / 2.0} 0 0" />
             <material name="grey" />
         </visual>
@@ -41,5 +46,5 @@
         <visual>
             <geometry>
-                <sphere radius="0.05" />
+                <sphere radius="${wheel_radius / 2.0}" />
             </geometry>
             <origin xyz="0 0 0" rpy="0 0 0" />
@@ -52,5 +57,5 @@
         <parent link="base_link" />
         <child link="right_wheel_link" />
-        <origin xyz="-0.15 -0.225 0" rpy="0 0 0" /> <!-- adding half of the cylinder height to the origin Y-->
+        <origin xyz="${-base_length / 4.0} ${-(base_width + wheel_length) / 2.0} 0" rpy="0 0 0" /> <!-- adding half of the cylinder height to the origin Y-->
         <axis xyz="0 1 0" />
     </joint>
@@ -58,5 +63,5 @@
         <parent link="base_link" />
         <child link="left_wheel_link" />
-        <origin xyz="-0.15 0.225 0" rpy="0 0 0" /> <!-- adding half of the cylinder height to the origin Y-->
+        <origin xyz="${-base_length / 4.0} ${(base_width + wheel_length) / 2.0} 0" rpy="0 0 0" /> <!-- adding half of the cylinder height to the origin Y-->
         <axis xyz="0 1 0" />
     </joint>
@@ -64,10 +69,10 @@
         <parent link="base_link" />
         <child link="caster_wheel_link" />
-        <origin xyz="0.2 0 -0.05" rpy="0 0 0" />
+        <origin xyz="${base_length / 3.0} 0 ${-wheel_radius / 2.0}" rpy="0 0 0" />
     </joint>
      <joint name="base_joint" type="fixed">
         <parent link="base_footprint_link" />
         <child link="base_link" />
-        <origin xyz="0 0 -0.1" rpy="0 0 0" />
+        <origin xyz="0 0 0.1" rpy="0 0 0" />
     </joint>
 </robot>

Commit message: xacro
split files for modular development

File: src/porter_bot_description/src/description/robot_description/porter_bot.urdf.xacro (robot description, xacro)
@@ -1,78 +1,5 @@
 <?xml version="1.0"?>
 <robot name="porter_bot" xmlns:xacro="http://wwww.ros.org/wiki/xacro">
-    <xacro:property name="base_length" value="0.6" />
-    <xacro:property name="base_width" value="0.4" />
-    <xacro:property name="base_height" value="0.2" />
-    <xacro:property name="wheel_radius" value="0.1" />
-    <xacro:property name="wheel_length" value="0.05" />
-    <material name="green">
-        <color rgba="0.5 0 0 1" />
-    </material>
-     <material name="grey">
-        <color rgba="0.5 0.5 0.5 1" />
-    </material>
-    <link name="base_link">
-        <visual>
-            <geometry>
-                <!--  <box size="0.157 0.073 0.055" />  -->
-                <box size="${base_length} ${base_width} ${base_height}" />
-            </geometry>
-            <!--  <origin xyz="0 0 0.0275" rpy="0 0 0" /> -->
-            <origin xyz="0 0 ${base_height / 2.0}" rpy="0 0 0" />
-            <material name="green" />
-        </visual>
-    </link>
-    <link name="right_wheel_link">
-        <visual>
-            <geometry>
-                <!-- <cylinder radius="0.03" length="0.007" /> -->
-                <cylinder radius="${wheel_radius}" length="${wheel_length}" />
-            </geometry>
-            <origin xyz="0 0 0" rpy="${pi / 2.0} 0 0" />
-            <material name="grey" />
-        </visual>
-    </link>
-     <link name="left_wheel_link">
-        <visual>
-            <geometry>
-                <!-- <cylinder radius="0.03" length="0.007" /> -->
-                <cylinder radius="${wheel_radius}" length="${wheel_length}" />
-            </geometry>
-            <origin xyz="0 0 0" rpy="${pi / 2.0} 0 0" />
-            <material name="grey" />
-        </visual>
-    </link>
-     <link name="caster_wheel_link">
-        <visual>
-            <geometry>
-                <sphere radius="${wheel_radius / 2.0}" />
-            </geometry>
-            <origin xyz="0 0 0" rpy="0 0 0" />
-            <material name="grey" />
-        </visual>
-    </link>
-     <link name="base_footprint_link">
-    </link>
-    <joint name="base_right_wheel_joint" type="continuous">
-        <parent link="base_link" />
-        <child link="right_wheel_link" />
-        <origin xyz="${-base_length / 4.0} ${-(base_width + wheel_length) / 2.0} 0" rpy="0 0 0" /> <!-- adding half of the cylinder height to the origin Y-->
-        <axis xyz="0 1 0" />
-    </joint>
-    <joint name="base_left_wheel_joint" type="continuous">
-        <parent link="base_link" />
-        <child link="left_wheel_link" />
-        <origin xyz="${-base_length / 4.0} ${(base_width + wheel_length) / 2.0} 0" rpy="0 0 0" /> <!-- adding half of the cylinder height to the origin Y-->
-        <axis xyz="0 1 0" />
-    </joint>
-    <joint name="base_caster_wheel_joint" type="fixed">
-        <parent link="base_link" />
-        <child link="caster_wheel_link" />
-        <origin xyz="${base_length / 3.0} 0 ${-wheel_radius / 2.0}" rpy="0 0 0" />
-    </joint>
-     <joint name="base_joint" type="fixed">
-        <parent link="base_footprint_link" />
-        <child link="base_link" />
-        <origin xyz="0 0 0.1" rpy="0 0 0" />
-    </joint>
+    <xacro:include filename="$(find porter_bot_description)/src/description/robot_description/common_properties.xacro" />
+    <xacro:include filename="$(find porter_bot_description)/src/description/robot_description/mobile_base.xacro" />
 </robot>

Commit message: combine the robots
arm and base together

File: src/porter_bot_description/src/description/robot_description/porter_bot.urdf.xacro (robot description, xacro)
@@ -4,4 +4,12 @@
     <xacro:include filename="$(find porter_bot_description)/src/description/robot_description/mobile_base.xacro" />
     <xacro:include filename="$(find porter_bot_description)/src/description/robot_description/mobile_base_gazebo.xacro" />
-    <xacro:include filename="$(find porter_bot_description)/src/description/robot_description/camera.xacro" />
+    <xacro:include filename="$(find porter_bot_description)/src/description/robot_description/arm.xacro" />
+    <xacro:include filename="$(find porter_bot_description)/src/description/robot_description/arm_gazebo.xacro" />
+     <joint name="mobile_base_arm_joint" type="fixed">
+        <parent link="base_link" />
+        <child link="arm_base_link" />
+        <origin xyz="${base_length/4.0} 0 ${base_height}" rpy="0 0 0" />
+    </joint>
+<!--     <xacro:include filename="$(find porter_bot_description)/src/description/robot_description/camera.xacro" />
+ -->
 </robot>
